File: pcb/usdx_smd.sch (EAGLE design)
At the start: 70 parts, among them IC1 MEGA8-AI, IC2 TL072P, IC4 REG1117, IC5 REG1117, IC6 74ACT00N, J2 JW-PJ-307-3, J3 JW-PJ-307-3, Q1 BS170, Q2 BS170, Q3 BS170, SW1 EC12E_SW, U1 Si5351A-B-GT, X1 1-227161-7, X2 27MHz, X3 CRYSTALS-NOGND-HC49

Commit message: Schematics maybe complete.
Parts:
- added C24: (no value), rcl:CPOL-EUCT7343
- added C25: 10n, rcl:C-EUC1206K
- added C26: 100n, rcl:C-EUC0603K
- added R26: 470, rcl:R-EU_M1206
- added R27, R28, R29: 10k, rcl:R-EU_M1206
- J2, J3: value JW-PJ-307-3 -> JW-PJ-307-5; device audioconn:JW-PJ-307-3 -> audioconn:JW-PJ-307-5
Connections:
- new net +5V_A: R29.2
- new net AUDIO_OUT: IC1.PB1(OC1A), R26.1
- new net MIC_IN: IC1.PB4(MISO)
- new net N$28: C26.2, R27.2, R28.1
- new net N$32: C25.2, C26.1, J3.4, J3.5, R29.1
- new net N$33: C24.-, J2.2, J2.3, J2.4, J2.5
- new net N$35: C24.+, R26.2
- new net PTT: IC1.PB5(SCK), J3.2, J3.3
- net AREF: now also R27.1
- net GND: now also C25.1, J2.1, J3.1, R28.2

Commit message: Schematics 99%, placing started.
Parts:
- removed U$1: FST3253, FST3253:FST3253
- removed U1: Si5351A-B-GT, microbuilder:SI5351A
- added C27: 100n, rcl:C-EUC0603K
- added C28, C29: 10n, rcl:C-EUC0603K
- added IC3: REG1117, burr-brown:REG1117
- added IC7: 74ACT00N, 74xx-eu:74ACT00N
- added Q4: BS170, transistor-small-signal:BS170
- added R30: 1k, rcl:R-EU_R1206
- C5: value (none) -> 10n
- IC2: value TL072P -> REG1117; device linear:TL072P -> burr-brown:REG1117
- IC4: value REG1117 -> Si5351A-B-GT; device burr-brown:REG1117 -> microbuilder:SI5351A
- IC5: value REG1117 -> FST3253; device burr-brown:REG1117 -> FST3253:FST3253
- IC6: value 74ACT00N -> TL072P; device 74xx-eu:74ACT00N -> linear:TL072P
- R22: value 1k -> FB; device rcl:R-EU_M1206 -> rcl:R-EU_R1206
Connections:
- removed net N$20: C17.1
- new net N$31: IC1.AVCC, R22.2
- new net RXS: C17.1, Q4.S, R30.2
- net +3V3: now also IC3.VOUT, IC4.VDD, IC4.VDDO; no longer IC5.VOUT, U1.VDD, U1.VDDO
- net +5V: now also C27.1, IC2.VOUT, IC3.VIN, IC5.VCC, IC6P.V+, IC7D.I0, IC7D.I1, IC7P.VCC, R22.1; no longer IC1.AVCC, IC2P.V+, IC4.VOUT, IC5.VIN, IC6D.I0, IC6D.I1, IC6P.VCC, U$1.VCC
- net CLK0: now also IC4.CLK0, IC5.S0; no longer U$1.S0, U1.CLK0
- net CLK1: now also IC4.CLK1, IC5.S1; no longer U$1.S1, U1.CLK1
- net CLK2: now also IC4.CLK2, IC7B.I1; no longer IC6B.I1, U1.CLK2
- net GND: now also C27.2, C28.1, IC2.GND, IC3.GND, IC5.OE1/, IC5.OE2/, IC6P.V-, IC7P.GND, R30.1; no longer IC2P.V-, IC6P.GND, U$1.GND, U$1.OE1/, U$1.OE2/, U1.GND
- net N$10: now also IC6B.+IN; no longer IC2B.+IN
- net N$11: now also IC6B.-IN; no longer IC2B.-IN
- net N$14: now also IC5.2B3; no longer U$1.2B3
- net N$15: now also IC5.2B2; no longer U$1.2B2
- net N$16: now also IC6A.OUT; no longer IC2A.OUT
- net N$17: now also IC5.2B4; no longer U$1.2B4
- net N$18: now also IC6B.OUT; no longer IC2B.OUT
- net N$19: now also IC5.2B1; no longer U$1.2B1
- net N$2: now also C29.1, Q4.D; no longer IC6A.I0, IC6A.I1
- net N$25: now also IC5.2A; no longer U$1.1A
- net N$3: now also IC6A.+IN; no longer IC2A.+IN
- net N$4: now also IC4.XB; no longer U1.XB
- net N$5: now also IC4.XA; no longer U1.XA
- net N$6: now also IC7A.O, IC7B.I0; no longer IC6A.O, IC6B.I0
- net N$7: now also IC7B.O, IC7C.I0, IC7C.I1; no longer IC6B.O, IC6C.I0, IC6C.I1
- net N$8: now also IC6A.-IN; no longer IC2A.-IN
- net N$9: now also IC7C.O; no longer IC6C.O
- net RD: now also C29.2
- net SCL: now also IC4.SCL; no longer U1.SCL
- net SDA: now also IC4.SDA; no longer U1.SDA
- net TX: now also C28.2, IC1.PB0(ICP), IC7A.I0, IC7A.I1, Q4.G
- net VCC: now also IC2.VIN; no longer IC4.VIN
Other:
- moved on the sheet: C17, C7, R16, R22

Commit message: Much much routing
Parts:
- removed J1: (no value), con-jack:DCJ0303
- removed JP2: (no value), pinhead:PINHD-1X4
- removed R20: 10k, rcl:R-TRIMMT93YA
- added C30: 100n, rcl:C-EUC0603K
- added C31: (no value), rcl:C-EUC0603K
- added CF1-A, CF1-B, CF2-A, CF2-B, CF3-A, CF3-B, CF4-A, CF4-B, CF5-A, CF5-B, CF6-A, CF6-B: (no value), rcl:C-EU025-024X044
- added H1, H2, H3, H4: MOUNT-PAD-ROUND3.2, holes:MOUNT-PAD-ROUND3.2
- added JP3, JP4: (no value), pinhead:PINHD-1X2
- added K1, K2: TQ2SA-L2-5V, relay:TQ2SA-L2-5V
- added L1-A, L1-B, L2-A, L2-B: T37, inductor:T37
- added R31, R32, R33, R34: 1k, rcl:R-EU_R1206
- added R35: 1k, rcl:R-EU_M1206
- added R36: (no value), rcl:R-TRIMM3374
- added T1, T2: (no value), transistor:-NPN-SOT23-EBC
- added U$5: FT37-43, inductor:T37
- C17, C28, C29: device rcl:C-EUC0603K -> rcl:C-EUC1206K
- JP1: device pinhead:PINHD-1X4 -> pinhead:PINHD-2X3
- X1: value 1-227161-7 -> BU-SMA-H; device con-coax:1-227161-7 -> con-coax:BU-SMA-H
Connections:
- removed net +12V: JP2.1
- removed net N$28: C26.2, R27.2, R28.1
- removed net N$35: C24.+, R26.2
- removed net RD: C29.2, JP2.3
- removed net TD: Q1.D, Q2.D, Q3.D
- new net AVCC: C6.1, IC1.AVCC, R22.2
- new net MOSI: IC1.PB3(MOSI/OC2), JP1.4
- new net N$20: K1R.-, K2R.-, T1.C
- new net N$34: JP3.1, JP4.2
- new net N$36: R31.1, T1.B
- new net N$37: R32.1, T2.B
- new net N$40: K11.P, X1.1
- new net N$44: K22.P
- new net N$46: CF5-A.1, CF6-A.1, K11.S, K12.O, L2-A.1
- new net N$47: CF2-A.2, CF3-A.2, CF4-A.2, CF5-A.2, L2-A.2
- new net N$48: CF5-B.1, CF6-B.1, K11.O, K12.S, L2-B.1
- new net N$49: CF2-B.2, CF3-B.2, CF4-B.2, CF5-B.2, L2-B.2
- new net N$50: CF2-B.1, CF3-B.1, L1-B.1
- new net N$51: CF2-A.1, CF3-A.1, L1-A.1
- new net N$52: CF1-A.1, K21.O, K22.S, L1-A.2
- new net N$53: CF1-B.1, K21.S, K22.O, L1-B.2
- new net PC2: IC1.PC2(ADC2)
- new net PD5: IC1.PD5(T1)
- new net RELAY1: IC1.ADC6, R31.2, R34.1
- new net RELAY2: IC1.ADC7, R32.2, R33.1
- new net SS: IC1.PB2(SS/OC1B)
- new net TRD: C29.2, Q1.D, Q2.D, Q3.D, U$5.1
- net +5V: now also JP1.2, K1R.+, K1S.+, K2R.+, K2S.+, R35.1; no longer C6.1
- net +5V_A: now also C31.1, R35.2
- net AUDIO_OUT: now also C24.+; no longer R26.1
- net GND: now also C30.2, C31.2, CF1-A.2, CF1-B.2, CF4-A.1, CF4-B.1, CF6-A.2, CF6-B.2, JP1.6, JP4.1, K12.P, K21.P, R33.2, R34.2, T1.E, T2.E; no longer J1.2, J1.3, JP1.1, JP1.2, JP2.4
- net LCD_CONTR: now also R36.S; no longer R20.S
- net LCD_VCC: now also R36.A; no longer R20.A
- net MIC_IN: now also C26.2, JP1.1, R27.2, R28.1
- net N$22: now also K1S.-, K2S.-, T2.C; no longer JP1.3, JP1.4, X1.1
- net N$27: now also R36.E; no longer R20.E
- net N$31: now also C24.-, R26.1; no longer IC1.AVCC, R22.2
- net N$33: now also R26.2; no longer C24.-
- net PTT: now also JP1.3
- net RESET: now also JP1.5
- net TX: no longer JP2.2
- net VCC: now also C30.1, JP3.2, U$5.2; no longer J1.1
